File: renovation_ssi_2001/renovation_ssi_2001.kicad_pcb (KiCad board)
At the start: 2 copper layers, 134.6 x 105.4 mm, 93 parts, among them J1 KLPX-0848A-2-B, J2 DB15_Female, J4 Bus_ISA_8bit, J5 Pins_02x04, J6 Pins_02x03, J7 SID_Socket, Q1 PN2222A, Q2 PN2222A, U1 74LS74, U10 74LS138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

Commit message: corrections and improvements
Parts:
- added C21: 100nF, Capacitor_SMD:C_0603_1608Metric, F.Cu at (165.7, 65.4)
- moved C17 3.19 mm to (161.3, 67.9)
- moved R10 3.18 mm to (162.6, 65.4)
- moved R9 3.18 mm to (159.4, 65.4)
- moved R18 1.52 mm to (165.7, 68.6)
- moved J4 0.64 mm to (198.1, 127.6)
Connections:
- U12 pad 39: /LOWPASS -> Net-(U12-Pad39)
- U12 pad 40: Net-(U12-Pad40) -> /LOWPASS
Routing:
- net +5V: track 596.1 -> 573.4 mm, vias 1 -> 3
- net GND: track 747.5 -> 741.5 mm, vias 3 -> 2
- net /OSC: track 70.8 -> 74.6 mm
- net Net-(R10-Pad1): track 3.72 -> 6.49 mm
- net /SID_D7: track 51.1 -> 52.9 mm
- net /ATTENUATOR: track 8.79 -> 10.3 mm
- net /SID_AUDIO_OUT: track 60.3 -> 59.0 mm
- net /SID_D6: track 43.7 -> 44.8 mm
- net /SID_D0: track 22.9 -> 23.8 mm
- net +12V: track 125.3 -> 124.5 mm
- net /LOWPASS: track 2.91 -> 3.45 mm
Other:
- board size 134.6 x 105.4 mm -> 134.6 x 106.4 mm

Commit message: fill in some component values, add pad to simplify fast ISA mod, adjust mounting hole positions
Parts:
- added TP1: TestPoint, TestPoint:TestPoint_Pad_1.5x1.5mm, F.Cu at (105.4, 52.1)
- C20: value C -> 100nF
- C7: value C -> DNP
- R7: value R -> 100
- moved H2 0.40 mm to (218.8, 60.8)
- moved H3 0.40 mm to (218.8, 117.3)
Changed lines of the file:
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@@
     (tracks 1238)
     (zones 0)
-    (modules 94)
+    (modules 95)
     (nets 171)
   )
@@
   (title_block
     (title "RENOVATION SSI-2001")
-    (date 2020-03-08)
+    (date 2020-03-10)
     (company "Benedikt Freisen")
     (comment 4 "INNOVATION SSI-2001 replica that can be built without vintage components")
@@
     (add_net GND)
   )
+  (module TestPoint:TestPoint_Pad_1.5x1.5mm (layer F.Cu)
+    (at 105.41 52.07)
+    (descr "SMD rectangular pad as test Point, square 1.5mm side length")
+    (tags "test point SMD pad rectangle square")
+    (attr virtual)
+    (fp_text reference TP1 (at 0 -1.648) (layer F.SilkS) hide
+      (effects (font (size 1 1) (thickness 0.15)))
+    )
+    (fp_text value TestPoint (at 0 1.75) (layer F.Fab)
+      (effects (font (size 1 1) (thickness 0.15)))
+    )
+    (fp_text user %R (at 0 -1.65) (layer F.Fab)
+      (effects (font (size 1 1) (thickness 0.15)))
+    )
+    (fp_line (start -0.95 -0.95) (end 0.95 -0.95) (layer F.SilkS) (width 0.12))
+    (fp_line (start 0.95 -0.95) (end 0.95 0.95) (layer F.SilkS) (width 0.12))
+    (fp_line (start 0.95 0.95) (end -0.95 0.95) (layer F.SilkS) (width 0.12))
+    (fp_line (start -0.95 0.95) (end -0.95 -0.95) (layer F.SilkS) (width 0.12))
+    (fp_line (start -1.25 -1.25) (end 1.25 -1.25) (layer F.CrtYd) (width 0.05))
+    (fp_line (start -1.25 -1.25) (end -1.25 1.25) (layer F.CrtYd) (width 0.05))
+    (fp_line (start 1.25 1.25) (end 1.25 -1.25) (layer F.CrtYd) (width 0.05))
+    (fp_line (start 1.25 1.25) (end -1.25 1.25) (layer F.CrtYd) (width 0.05))
+    (pad 1 smd rect (at 0 0) (size 1.5 1.5) (layers F.Cu F.Mask)
+      (net 134 /ACCESS))
+  )
   (module Capacitor_Tantalum_SMD:CP_EIA-3528-21_Kemet-B (layer F.Cu)
     (at 161.29 67.945)
@@
       (effects (font (size 1 1) (thickness 0.15)))
     )
-    (fp_text value C (at 1.25 2.3) (layer F.Fab)
+    (fp_text value DNP (at 1.25 2.3) (layer F.Fab)
       (effects (font (size 1 1) (thickness 0.15)))
     )
@@
   )
   (module SSI_2001:MountingHole_3.2mm_M3 (layer F.Cu)
-    (at 218.44 117.475)
+    (at 218.821 117.348)
     (descr "Mounting Hole 3.2mm, no annular, M3")
     (tags "mounting hole 3.2mm no annular m3")
@@
       (effects (font (size 1 1) (thickness 0.15)))
     )
-    (fp_text value MountingHole (at 0 4.2) (layer F.Fab)
+    (fp_text value MountingHole (at -0.635 4.191) (layer F.Fab)
       (effects (font (size 1 1) (thickness 0.15)))
     )
+    (fp_circle (center 0 0) (end 3.45 0) (layer F.CrtYd) (width 0.05))
+    (fp_circle (center 0 0) (end 3.2 0) (layer Cmts.User) (width 0.15))
     (fp_text user %R (at 0.3 0) (layer F.Fab)
       (effects (font (size 1 1) (thickness 0.15)))
     )
-    (fp_circle (center 0 0) (end 3.2 0) (layer Cmts.User) (width 0.15))
-    (fp_circle (center 0 0) (end 3.45 0) (layer F.CrtYd) (width 0.05))
     (pad "" np_thru_hole circle (at 0 0) (size 3.2 3.2) (drill 3.2) (layers *.Cu *.Mask)
       (solder_mask_margin 0.635))
   )
   (module SSI_2001:MountingHole_3.2mm_M3 (layer F.Cu)
-    (at 218.44 60.96)
+    (at 218.821 60.833)
     (descr "Mounting Hole 3.2mm, no annular, M3")
     (tags "mounting hole 3.2mm no annular m3")
@@
       (effects (font (size 1 1) (thickness 0.15)))
     )
-    (fp_text value MountingHole (at 0 -4.445) (layer F.Fab)
+    (fp_text value MountingHole (at -0.635 -4.445) (layer F.Fab)
       (effects (font (size 1 1) (thickness 0.15)))
     )
+    (fp_circle (center 0 0) (end 3.45 0) (layer F.CrtYd) (width 0.05))
+    (fp_circle (center 0 0) (end 3.2 0) (layer Cmts.User) (width 0.15))
     (fp_text user %R (at 0.3 0) (layer F.Fab)
       (effects (font (size 1 1) (thickness 0.15)))
     )
-    (fp_circle (center 0 0) (end 3.2 0) (layer Cmts.User) (width 0.15))
-    (fp_circle (center 0 0) (end 3.45 0) (layer F.CrtYd) (width 0.05))
     (pad "" np_thru_hole circle (at 0 0) (size 3.2 3.2) (drill 3.2) (layers *.Cu *.Mask)
       (solder_mask_margin 0.635))
@@
       (effects (font (size 1 1) (thickness 0.15)))
     )
-    (fp_text value SolderJumper_2_Open (at 0 1.9) (layer F.Fab)
+    (fp_text value SolderJumper_2_Open (at 2.54 0 90) (layer F.Fab)
       (effects (font (size 1 1) (thickness 0.15)))
     )
-    (fp_arc (start 0.7 -0.3) (end 1.4 -0.3) (angle -90) (layer F.SilkS) (width 0.12))
-    (fp_arc (start 0.7 0.3) (end 0.7 1) (angle -90) (layer F.SilkS) (width 0.12))
-    (fp_arc (start -0.7 0.3) (end -1.4 0.3) (angle -90) (layer F.SilkS) (width 0.12))
-    (fp_arc (start -0.7 -0.3) (end -0.7 -1) (angle -90) (layer F.SilkS) (width 0.12))
-    (fp_line (start -1.4 0.3) (end -1.4 -0.3) (layer F.SilkS) (width 0.12))
-    (fp_line (start 0.7 1) (end -0.7 1) (layer F.SilkS) (width 0.12))
-    (fp_line (start 1.4 -0.3) (end 1.4 0.3) (layer F.SilkS) (width 0.12))
-    (fp_line (start -0.7 -1) (end 0.7 -1) (layer F.SilkS) (width 0.12))
-    (fp_line (start -1.65 -1.25) (end 1.65 -1.25) (layer F.CrtYd) (width 0.05))
-    (fp_line (start -1.65 -1.25) (end -1.65 1.25) (layer F.CrtYd) (width 0.05))
-    (fp_line (start 1.65 1.25) (end 1.65 -1.25) (layer F.CrtYd) (width 0.05))
     (fp_line (start 1.65 1.25) (end -1.65 1.25) (layer F.CrtYd) (width 0.05))
-    (pad 1 smd custom (at -0.65 0) (size 1 0.5) (layers F.Cu F.Mask)
-      (net 135 /~ACCESS) (zone_connect 2)
+    (fp_line (start 1.65 1.25) (end 1.65 -1.25) (layer F.CrtYd) (width 0.05))
+    (fp_line (start -1.65 -1.25) (end -1.65 1.25) (layer F.CrtYd) (width 0.05))
+    (fp_line (start -1.65 -1.25) (end 1.65 -1.25) (layer F.CrtYd) (width 0.05))
+    (fp_line (start -0.7 -1) (end 0.7 -1) (layer F.SilkS) (width 0.12))
+    (fp_line (start 1.4 -0.3) (end 1.4 0.3) (layer F.SilkS) (width 0.12))
+    (fp_line (start 0.7 1) (end -0.7 1) (layer F.SilkS) (width 0.12))
+    (fp_line (start -1.4 0.3) (end -1.4 -0.3) (layer F.SilkS) (width 0.12))
+    (fp_arc (start -0.7 -0.3) (end -0.7 -1) (angle -90) (layer F.SilkS) (width 0.12))
+    (fp_arc (start -0.7 0.3) (end -1.4 0.3) (angle -90) (layer F.SilkS) (width 0.12))
+    (fp_arc (start 0.7 0.3) (end 0.7 1) (angle -90) (layer F.SilkS) (width 0.12))
+    (fp_arc (start 0.7 -0.3) (end 1.4 -0.3) (angle -90) (layer F.SilkS) (width 0.12))
+    (pad 2 smd custom (at 0.65 0) (size 1 0.5) (layers F.Cu F.Mask)
+      (net 169 /~CS) (zone_connect 2)
       (options (clearance outline) (anchor rect))
       (primitives
@@
         (gr_circle (center 0 -0.25) (end 0.5 -0.25) (width 0))
         (gr_poly (pts
-           (xy 0 -0.75) (xy 0.5 -0.75) (xy 0.5 0.75) (xy 0 0.75)) (width 0))
+           (xy 0 -0.75) (xy -0.5 -0.75) (xy -0.5 0.75) (xy 0 0.75)) (width 0))
       ))
-    (pad 2 smd custom (at 0.65 0) (size 1 0.5) (layers F.Cu F.Mask)
-      (net 169 /~CS) (zone_connect 2)
+    (pad 1 smd custom (at -0.65 0) (size 1 0.5) (layers F.Cu F.Mask)
+      (net 135 /~ACCESS) (zone_connect 2)
       (options (clearance outline) (anchor rect))
       (primitives
@@
         (gr_circle (center 0 -0.25) (end 0.5 -0.25) (width 0))
         (gr_poly (pts
-           (xy 0 -0.75) (xy -0.5 -0.75) (xy -0.5 0.75) (xy 0 0.75)) (width 0))
+           (xy 0 -0.75) (xy 0.5 -0.75) (xy 0.5 0.75) (xy 0 0.75)) (width 0))
       ))
   )
@@
       (effects (font (size 1 1) (thickness 0.15)))
     )
-    (fp_text value C (at 0 1.43) (layer F.Fab)
+    (fp_text value 100nF (at 0 1.43) (layer F.Fab)
       (effects (font (size 1 1) (thickness 0.15)))
     )
@@
       (effects (font (size 1 1) (thickness 0.15)))
     )
-    (fp_text value R (at 0 1.43) (layer F.Fab)
+    (fp_text value 100 (at 0 1.43) (layer F.Fab)
       (effects (font (size 1 1) (thickness 0.15)))
     )

Commit message: correct configuration resistor values for the voltage regulator
Parts:
- R10: value 1k -> 180
- R9: value 10k -> 110
Changed lines of the file:
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@@
   (title_block
     (title "RENOVATION SSI-2001")
-    (date 2020-03-10)
+    (date 2020-03-13)
     (company "Benedikt Freisen")
     (comment 4 "INNOVATION SSI-2001 replica that can be built without vintage components")
@@
       (effects (font (size 1 1) (thickness 0.15)))
     )
-    (fp_text value 1k (at 0 -1.27) (layer F.Fab)
+    (fp_text value 180 (at 0 -1.27) (layer F.Fab)
       (effects (font (size 1 1) (thickness 0.15)))
     )
@@
       (effects (font (size 1 1) (thickness 0.15)))
     )
-    (fp_text value 10k (at 0 -1.27) (layer F.Fab)
+    (fp_text value 110 (at 0 -1.27) (layer F.Fab)
       (effects (font (size 1 1) (thickness 0.15)))
     )
